Commit message: taskD

File: nuturtle_description/urdf/turtlebot3_burger.urdf.xacro (robot description, xacro)
@@ -6,4 +6,5 @@
   <xacro:property name="R" value="${robot_param['R']}" />
   <xacro:property name="W" value="${robot_param['W']}" />
+  <xacro:property name="C_R" value="${robot_param['C_R']}" />
   <xacro:arg name="color" default="black"/>
   <!-- <xacro:property name="color" value="$(arg color)" /> -->
@@ -25,5 +26,5 @@
       <origin xyz="-0.032 0 0.070" rpy="0 0 0"/>
       <geometry>
-        <box size="0.140 0.140 0.143"/>
+        <cylinder length="0.24" radius="${C_R}"/>
       </geometry>
     </collision>

Commit message: got blue robot in rviz

File: nuturtle_description/urdf/turtlebot3_burger.urdf.xacro (robot description, xacro)
@@ -9,11 +9,11 @@
   <xacro:arg name="color" default="black"/>
   <!-- <xacro:property name="color" value="$(arg color)" /> -->
-  <link name="$(arg color):base_footprint"/>
-  <joint name="$(arg color):base_joint" type="fixed">
-    <parent link="$(arg color):base_footprint"/>
-    <child link="$(arg color):base_link"/>
+  <link name="$(arg color)-base_footprint"/>
+  <joint name="$(arg color)-base_joint" type="fixed">
+    <parent link="$(arg color)-base_footprint"/>
+    <child link="$(arg color)-base_link"/>
     <origin xyz="0.0 0.0 0.010" rpy="0 0 0"/>
   </joint>
-  <link name="$(arg color):base_link">
+  <link name="$(arg color)-base_link">
     <visual>
       <origin xyz="-0.032 0 0.0" rpy="0 0 0"/>
@@ -37,11 +37,11 @@
     </inertial>
   </link>
-  <joint name="$(arg color):wheel_left_joint" type="continuous">
-    <parent link="$(arg color):base_link"/>
-    <child link="$(arg color):wheel_left_link"/>
+  <joint name="$(arg color)-wheel_left_joint" type="continuous">
+    <parent link="$(arg color)-base_link"/>
+    <child link="$(arg color)-wheel_left_link"/>
     <origin xyz="0.0 ${W} 0.023" rpy="-1.57 0 0"/>
     <axis xyz="0 0 1"/>
   </joint>
-  <link name="$(arg color):wheel_left_link">
+  <link name="$(arg color)-wheel_left_link">
     <visual>
       <origin xyz="0 0 0" rpy="1.57 0 0"/>
@@ -65,11 +65,11 @@
       </inertial>
   </link>
-  <joint name="$(arg color):wheel_right_joint" type="continuous">
-    <parent link="$(arg color):base_link"/>
-    <child link="$(arg color):wheel_right_link"/>
+  <joint name="$(arg color)-wheel_right_joint" type="continuous">
+    <parent link="$(arg color)-base_link"/>
+    <child link="$(arg color)-wheel_right_link"/>
     <origin xyz="0.0 -${W} 0.023" rpy="-1.57 0 0"/>
     <axis xyz="0 0 1"/>
   </joint>
-  <link name="$(arg color):wheel_right_link">
+  <link name="$(arg color)-wheel_right_link">
     <visual>
       <origin xyz="0 0 0" rpy="1.57 0 0"/>
@@ -93,10 +93,10 @@
       </inertial>
   </link>
-  <joint name="$(arg color):caster_back_joint" type="fixed">
-    <parent link="$(arg color):base_link"/>
-    <child link="$(arg color):caster_back_link"/>
+  <joint name="$(arg color)-caster_back_joint" type="fixed">
+    <parent link="$(arg color)-base_link"/>
+    <child link="$(arg color)-caster_back_link"/>
     <origin xyz="-0.081 0 -0.004" rpy="-1.57 0 0"/>
   </joint>
-  <link name="$(arg color):caster_back_link">
+  <link name="$(arg color)-caster_back_link">
     <collision>
       <origin xyz="0 0.001 0" rpy="0 0 0"/>
@@ -113,16 +113,16 @@
     </inertial>
   </link>
-  <joint name="$(arg color):imu_joint" type="fixed">
-    <parent link="$(arg color):base_link"/>
-    <child link="$(arg color):imu_link"/>
+  <joint name="$(arg color)-imu_joint" type="fixed">
+    <parent link="$(arg color)-base_link"/>
+    <child link="$(arg color)-imu_link"/>
     <origin xyz="-0.032 0 0.068" rpy="0 0 0"/>
   </joint>
-  <link name="$(arg color):imu_link"/>
-  <joint name="$(arg color):scan_joint" type="fixed">
-    <parent link="$(arg color):base_link"/>
-    <child link="$(arg color):base_scan"/>
+  <link name="$(arg color)-imu_link"/>
+  <joint name="$(arg color)-scan_joint" type="fixed">
+    <parent link="$(arg color)-base_link"/>
+    <child link="$(arg color)-base_scan"/>
     <origin xyz="-0.032 0 0.172" rpy="0 0 0"/>
   </joint>
-  <link name="$(arg color):base_scan">
+  <link name="$(arg color)-base_scan">
     <visual>
       <origin xyz="0 0 0.0" rpy="0 0 0"/>
